File: PCB/CAN.kicad_sch (KiCad schematic)
At the start: 7 parts, among them U6 SN65HVD232, U7 MCP2515-xST, Y2 Crystal_GND24

Commit message: fix: mark C28, C29, R24 as `+can`
Parts:
- C28, C29, R24: Config (none) -> +can
Changed lines of the file:
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@@
+      (effects (font (size 1.27 1.27)) hide)
+    )
+    (property "Config" "+can" (id 7) (at 154.94 109.22 90)
       (effects (font (size 1.27 1.27)) hide)
     )
@@
     )
     (property "Stock_PN" "C-603-27pF-50V-COG" (id 6) (at 238.125 99.06 0)
+      (effects (font (size 1.27 1.27)) hide)
+    )
+    (property "Config" "+can" (id 7) (at 238.125 99.06 90)
       (effects (font (size 1.27 1.27)) hide)
     )
@@
       (effects (font (size 1.27 1.27)) hide)
     )
+    (property "Config" "+can" (id 7) (at 238.125 106.68 90)
+      (effects (font (size 1.27 1.27)) hide)
+    )
