File: PCB/Power.kicad_sch (KiCad schematic)
At the start: 11 parts, among them J7 Conn_01x06_Male, J8 Conn_01x06_Male, U3 DRV8300DRGER, U4 INA180A4

Commit message: fix(power): update PNs for R18 shunt
Parts:
- R18: Digikey 738-CSM2512FT33L0CT-ND -> 1712-TLRP3A30DR003FTDGCT-ND; LCSC C2889925 -> C2889862; Part Number ARP2512GJR033 -> ARD2512GJR003; Stock_PN R-2512-.033-3W-5% -> R-2512-.003-3W-5%
Changed lines of the file:
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@@
       (effects (font (size 1.27 1.27)) hide)
     )
-    (property "LCSC" "C2889925" (id 4) (at 243.84 136.525 0)
+    (property "LCSC" "C2889862" (id 4) (at 243.84 136.525 0)
       (effects (font (size 1.27 1.27)) hide)
     )
-    (property "Stock_PN" "R-2512-.033-3W-5%" (id 5) (at 243.84 136.525 0)
+    (property "Stock_PN" "R-2512-.003-3W-5%" (id 5) (at 243.84 136.525 0)
       (effects (font (size 1.27 1.27)) hide)
     )
-    (property "Part Number" "ARP2512GJR033" (id 6) (at 243.84 136.525 0)
+    (property "Part Number" "ARD2512GJR003" (id 6) (at 243.84 136.525 0)
       (effects (font (size 1.27 1.27)) hide)
     )
-    (property "Digikey" "738-CSM2512FT33L0CT-ND" (id 7) (at 243.84 136.525 0)
+    (property "Digikey" "1712-TLRP3A30DR003FTDGCT-ND" (id 7) (at 243.84 136.525 0)
       (effects (font (size 1.27 1.27)) hide)
     )
