File: PCB/xESC2.kicad_pcb (KiCad board)
At the start: 4 copper layers, 49.5 x 29 mm, 90 parts, among them J1 Conn_01x09_Male, J10 Conn_02x02_Counter_Clockwise, J2 U254-051T-4BH83-F1S, J3 Conn_01x05_Male, J4 Conn_01x05_Male, J5 Conn_01x02, J6 Conn_02x02_Counter_Clockwise, J7 Conn_01x06_Male, J8 Conn_01x06_Male, J9 Conn_02x02_Counter_Clockwise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

Commit message: added .1uF for C2-C4
Parts:
- C2, C3, C4: value DNP -> .1uF
Changed lines of the file:
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@@
     )
   )
+  (property "git_version" "WIP")
   (net 0 "")
   (net 1 "Net-(Q1-Pad4)")
@@
     (descr "Capacitor SMD 0603 (1608 Metric), square (rectangular) end terminal, IPC_7351 nominal, (Body size source: IPC-SM-782 page 76, https://www.pcb-3d.com/wordpress/wp-content/uploads/ipc-sm-782a_amendment_1_and_2.pdf), generated with kicad-footprint-generator")
     (tags "capacitor")
-    (property "Config" "do not place")
+    (property "Config" "")
+    (property "Digikey" "1276-1935-1-ND")
+    (property "Part Number" "CL10B104KC8NNNC")
     (property "Sheetfile" "xESC2.kicad_sch")
     (property "Sheetname" "")
+    (property "Stock_PN" "C-603-.1uF-100V-X7R")
     (attr smd)
     (fp_text reference "C2" (at 0 -1.43 90) (layer "F.SilkS") hide
       (effects (font (size 1 1) (thickness 0.15)))
     )
-    (fp_text value "DNP" (at 0 1.43 90) (layer "F.Fab")
+    (fp_text value ".1uF" (at 0 1.43 90) (layer "F.Fab")
       (effects (font (size 1 1) (thickness 0.15)))
     )
@@
     (descr "Capacitor SMD 0603 (1608 Metric), square (rectangular) end terminal, IPC_7351 nominal, (Body size source: IPC-SM-782 page 76, https://www.pcb-3d.com/wordpress/wp-content/uploads/ipc-sm-782a_amendment_1_and_2.pdf), generated with kicad-footprint-generator")
     (tags "capacitor")
-    (property "Config" "do not place")
+    (property "Config" "")
+    (property "Digikey" "1276-1935-1-ND")
+    (property "Part Number" "CL10B104KC8NNNC")
     (property "Sheetfile" "xESC2.kicad_sch")
     (property "Sheetname" "")
+    (property "Stock_PN" "C-603-.1uF-100V-X7R")
     (attr smd)
     (fp_text reference "C3" (at 0 -1.43 90) (layer "F.SilkS") hide
       (effects (font (size 1 1) (thickness 0.15)))
     )
-    (fp_text value "DNP" (at 0 1.43 90) (layer "F.Fab")
+    (fp_text value ".1uF" (at 0 1.43 90) (layer "F.Fab")
       (effects (font (size 1 1) (thickness 0.15)))
     )
@@
     (descr "Capacitor SMD 0603 (1608 Metric), square (rectangular) end terminal, IPC_7351 nominal, (Body size source: IPC-SM-782 page 76, https://www.pcb-3d.com/wordpress/wp-content/uploads/ipc-sm-782a_amendment_1_and_2.pdf), generated with kicad-footprint-generator")
     (tags "capacitor")
-    (property "Config" "do not place")
+    (property "Config" "")
+    (property "Digikey" "1276-1935-1-ND")
+    (property "Part Number" "CL10B104KC8NNNC")
     (property "Sheetfile" "xESC2.kicad_sch")
     (property "Sheetname" "")
+    (property "Stock_PN" "C-603-.1uF-100V-X7R")
     (attr smd)
     (fp_text reference "C4" (at 0 -1.43 90) (layer "F.SilkS") hide
       (effects (font (size 1 1) (thickness 0.15)))
     )
-    (fp_text value "DNP" (at 0 1.43 90) (layer "F.Fab")
+    (fp_text value ".1uF" (at 0 1.43 90) (layer "F.Fab")
       (effects (font (size 1 1) (thickness 0.15)))
     )
@@
     (descr "SMD Crystal SERIES SMD3225/4 http://www.txccrystal.com/images/pdf/7m-accuracy.pdf, 3.2x2.5mm^2 package")
     (tags "SMD SMT crystal")
-    (property "Digikey" "50-ECS-80-12-33-JGN-CT-ND")
-    (property "Part Number" "ECS-80-12-33-JGN-TR")
+    (property "Digikey" "50-ECS-120-18-33-JGN-TR3CT-ND")
+    (property "Part Number" "ECS-120-18-33-JGN-TR3")
     (property "Sheetfile" "MCU.kicad_sch")
     (property "Sheetname" "MCU")
-    (property "Stock_PN" "Y-4-SMD-8MhHz")
+    (property "Stock_PN" "Y-1-SMD-12MhHz")
     (attr smd)
     (fp_text reference "Y1" (at 0 -2.45) (layer "F.SilkS") hide
@@
     (descr "Capacitor SMD 0603 (1608 Metric), square (rectangular) end terminal, IPC_7351 nominal, (Body size source: IPC-SM-782 page 76, https://www.pcb-3d.com/wordpress/wp-content/uploads/ipc-sm-782a_amendment_1_and_2.pdf), generated with kicad-footprint-generator")
     (tags "capacitor")
+    (property "Config" "+can")
     (property "Digikey" "311-1063-1-ND")
     (property "Part Number" "CC0603JRNPO9BN270")
@@
     (descr "Capacitor SMD 0603 (1608 Metric), square (rectangular) end terminal, IPC_7351 nominal, (Body size source: IPC-SM-782 page 76, https://www.pcb-3d.com/wordpress/wp-content/uploads/ipc-sm-782a_amendment_1_and_2.pdf), generated with kicad-footprint-generator")
     (tags "capacitor")
+    (property "Config" "+can")
     (property "Digikey" "311-1063-1-ND")
     (property "Part Number" "CC0603JRNPO9BN270")
@@
     (descr "Resistor SMD 0603 (1608 Metric), square (rectangular) end terminal, IPC_7351 nominal, (Body size source: IPC-SM-782 page 72, https://www.pcb-3d.com/wordpress/wp-content/uploads/ipc-sm-782a_amendment_1_and_2.pdf), generated with kicad-footprint-generator")
     (tags "resistor")
+    (property "Config" "+can")
     (property "Digikey" "311-10.0KHRCT-ND")
     (property "Part Number" "RC0603FR-0710KL")
